File: Keyboard_Scanner.brd (EAGLE design)
At the start: 48.3 x 47.8 mm, 3 parts

Commit message: Add files via upload
Parts:
- added E$4: (no value), oshw:OSHW_5MM
Changed lines of the file:
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@@
 <?xml version="1.0" encoding="utf-8"?>
 <!DOCTYPE eagle SYSTEM "eagle.dtd">
-<eagle version="8.2.2">
+<eagle version="9.2.2">
 <drawing>
 <settings>
-<setting alwaysvectorfont="no"/>
+<setting alwaysvectorfont="yes"/>
+<setting keepoldvectorfont="yes"/>
 <setting verticaltext="up"/>
 </settings>
@@
 <param name="dpMaxLengthDifference" value="10mm"/>
 <param name="dpGapFactor" value="2.5"/>
-<param name="checkGrid" value="0"/>
 <param name="checkAngle" value="0"/>
 <param name="checkFont" value="1"/>
 <param name="checkRestrict" value="1"/>
+<param name="checkStop" value="0"/>
+<param name="checkValues" value="0"/>
+<param name="checkNames" value="1"/>
+<param name="checkWireStubs" value="1"/>
+<param name="checkPolygonWidth" value="0"/>
 <param name="useDiameter" value="13"/>
 <param name="maxErrors" value="50"/>
@@
 </autorouter>
 <elements>
-<element name="E$1" library="Teensy_Combo" package="TEENSY_COMBO" value="" x="27.3812" y="31.369"/>
-<element name="E$2" library="FPC_Dual_front" package="FPC_DUAL" value="" x="27.94" y="10.16"/>
-<element name="E$3" library="FPC_Dual_back" package="FPC_DUAL_FRONT" value="" x="21.6408" y="10.0838"/>
+<element name="E$1" library="Teensy_Combo" package="TEENSY_COMBO" value="" x="27.3812" y="31.369" smashed="yes"/>
+<element name="E$2" library="FPC_Dual_front" package="FPC_DUAL" value="" x="27.94" y="10.16" smashed="yes"/>
+<element name="E$3" library="FPC_Dual_back" package="FPC_DUAL_FRONT" value="" x="21.6408" y="10.0838" smashed="yes"/>
+<element name="E$4" library="oshw" package="OSHW_5MM" value="" x="5.207" y="38.862" smashed="yes"/>
 </elements>
 <signals>
@@
 </signal>
 </signals>
+<mfgpreviewcolors>
+<mfgpreviewcolor name="soldermaskcolor" color="0xC8008000"/>
+<mfgpreviewcolor name="silkscreencolor" color="0xFFFEFEFE"/>
+<mfgpreviewcolor name="backgroundcolor" color="0xFF282828"/>
+<mfgpreviewcolor name="coppercolor" color="0xFFFFBF00"/>
+<mfgpreviewcolor name="substratecolor" color="0xFF786E46"/>
+</mfgpreviewcolors>
 </board>
 </drawing>
+<compatibility>
+<note version="6.3" minversion="6.2.2" severity="warning">
+Since Version 6.2.2 text objects can contain more than one line,
+which will not be processed correctly with this version.
+</note>
+</compatibility>
 </eagle>
