File: Example_Keyboards/Lenovo_ThinkPad_T61/Teensy 3p2/Lenovo_Scanner.brd (EAGLE design)
At the start: 49.8 x 49.8 mm, 9 parts

Commit message: Add files via upload
Parts:
- added E$10: (no value), oshw:OSHW_5MM
Changed lines of the file:
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@@
 <?xml version="1.0" encoding="utf-8"?>
 <!DOCTYPE eagle SYSTEM "eagle.dtd">
-<eagle version="8.2.2">
+<eagle version="9.2.2">
 <drawing>
 <settings>
 <setting alwaysvectorfont="yes"/>
+<setting keepoldvectorfont="yes"/>
 <setting verticaltext="up"/>
 </settings>
@@
 <param name="dpMaxLengthDifference" value="10mm"/>
 <param name="dpGapFactor" value="2.5"/>
-<param name="checkGrid" value="0"/>
 <param name="checkAngle" value="0"/>
 <param name="checkFont" value="1"/>
 <param name="checkRestrict" value="1"/>
+<param name="checkStop" value="0"/>
+<param name="checkValues" value="0"/>
+<param name="checkNames" value="1"/>
+<param name="checkWireStubs" value="1"/>
+<param name="checkPolygonWidth" value="0"/>
 <param name="useDiameter" value="13"/>
 <param name="maxErrors" value="50"/>
@@
 </autorouter>
 <elements>
-<element name="E$2" library="WM6787CT-ND" package="WM6787CT-ND" value="" x="11.7" y="41.3" populate="no" rot="R90"/>
-<element name="E$1" library="Teensy_3p2_min" package="TEENSY_3P2MIN" value="" x="33.4" y="30" rot="R270"/>
-<element name="E$3" library="SparkFun-Connectors" package="1X01" value="" x="2.4" y="18.8" populate="no"/>
-<element name="E$8" library="SparkFun-Connectors" package="1X02" value="" x="47.5" y="22.4" populate="no" rot="R90"/>
-<element name="E$7" library="SparkFun-Connectors" package="1X02" value="" x="47.5" y="9.7" populate="no" rot="R90"/>
-<element name="E$4" library="SparkFun-Connectors" package="1X05" value="" x="31.6" y="3.9" populate="no"/>
-<element name="E$5" library="SparkFun-Connectors" package="1X02" value="" x="2.4" y="42.6" populate="no"/>
-<element name="E$9" library="SparkFun-Connectors" package="1X02" value="" x="2.4" y="26" populate="no"/>
-<element name="E$6" library="SparkFun-Connectors" package="1X05" value="" x="47.5" y="32.5" populate="no" rot="R90"/>
+<element name="E$2" library="WM6787CT-ND" package="WM6787CT-ND" value="" x="11.7" y="41.3" populate="no" smashed="yes" rot="R90">
+<attribute name="NAME" x="7.9916" y="46.66" size="0.4064" layer="25" rot="R90"/>
+<attribute name="VALUE" x="13.1" y="49.2" size="0.6096" layer="27" rot="R90"/>
+</element>
+<element name="E$1" library="Teensy_3p2_min" package="TEENSY_3P2MIN" value="" x="33.4" y="30" smashed="yes" rot="R270"/>
+<element name="E$3" library="SparkFun-Connectors" package="1X01" value="" x="2.4" y="18.8" populate="no" smashed="yes">
+<attribute name="NAME" x="1.13" y="20.197" size="0.6096" layer="25" font="vector" ratio="20"/>
+<attribute name="VALUE" x="1.13" y="17.276" size="0.6096" layer="27" font="vector" ratio="20" align="top-left"/>
+</element>
+<element name="E$8" library="SparkFun-Connectors" package="1X02" value="" x="47.5" y="22.4" populate="no" smashed="yes" rot="R90">
+<attribute name="NAME" x="46.103" y="21.13" size="0.6096" layer="25" font="vector" ratio="20" rot="R90"/>
+<attribute name="VALUE" x="49.532" y="21.13" size="0.6096" layer="27" font="vector" ratio="20" rot="R90"/>
+</element>
+<element name="E$7" library="SparkFun-Connectors" package="1X02" value="" x="47.5" y="9.7" populate="no" smashed="yes" rot="R90">
+<attribute name="NAME" x="46.103" y="8.43" size="0.6096" layer="25" font="vector" ratio="20" rot="R90"/>
+<attribute name="VALUE" x="49.532" y="8.43" size="0.6096" layer="27" font="vector" ratio="20" rot="R90"/>
+</element>
+<element name="E$4" library="SparkFun-Connectors" package="1X05" value="" x="31.6" y="3.9" populate="no" smashed="yes">
+<attribute name="NAME" x="30.33" y="5.297" size="0.6096" layer="25" font="vector" ratio="20"/>
+<attribute name="VALUE" x="30.33" y="1.868" size="0.6096" layer="27" font="vector" ratio="20"/>
+</element>
+<element name="E$5" library="SparkFun-Connectors" package="1X02" value="" x="2.4" y="42.6" populate="no" smashed="yes">
+<attribute name="NAME" x="1.13" y="43.997" size="0.6096" layer="25" font="vector" ratio="20"/>
+<attribute name="VALUE" x="1.13" y="40.568" size="0.6096" layer="27" font="vector" ratio="20"/>
+</element>
+<element name="E$9" library="SparkFun-Connectors" package="1X02" value="" x="2.4" y="26" populate="no" smashed="yes">
+<attribute name="NAME" x="1.13" y="27.397" size="0.6096" layer="25" font="vector" ratio="20"/>
+<attribute name="VALUE" x="1.13" y="23.968" size="0.6096" layer="27" font="vector" ratio="20"/>
+</element>
+<element name="E$6" library="SparkFun-Connectors" package="1X05" value="" x="47.5" y="32.5" populate="no" smashed="yes" rot="R90">
+<attribute name="NAME" x="46.103" y="31.23" size="0.6096" layer="25" font="vector" ratio="20" rot="R90"/>
+<attribute name="VALUE" x="49.532" y="31.23" size="0.6096" layer="27" font="vector" ratio="20" rot="R90"/>
+</element>
+<element name="E$10" library="oshw" package="OSHW_5MM" value="" x="5.6" y="10.4" smashed="yes"/>
 </elements>
 <signals>
@@
 </signal>
 </signals>
+<mfgpreviewcolors>
+<mfgpreviewcolor name="soldermaskcolor" color="0xC8008000"/>
+<mfgpreviewcolor name="silkscreencolor" color="0xFFFEFEFE"/>
+<mfgpreviewcolor name="backgroundcolor" color="0xFF282828"/>
+<mfgpreviewcolor name="coppercolor" color="0xFFFFBF00"/>
+<mfgpreviewcolor name="substratecolor" color="0xFF786E46"/>
+</mfgpreviewcolors>
 </board>
 </drawing>
+<compatibility>
+<note version="6.3" minversion="6.2.2" severity="warning">
+Since Version 6.2.2 text objects can contain more than one line,
+which will not be processed correctly with this version.
+</note>
+</compatibility>
 </eagle>
