File: Example_Keyboards/Lenovo_ThinkPad_T61/Teensy LC/Eagle/T61_LC_Scanner.brd (EAGLE design)
At the start: 49.8 x 49.8 mm, 14 parts, among them J1 WM6787CT-ND, Q1 BSS138, Q2 BSS138, U1 TEENSY_LC, U2 TLV810SDBZT

Commit message: Add files via upload
Parts:
- added U$1: (no value), oshw:OSHW_5MM
Changed lines of the file:
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@@
 <?xml version="1.0" encoding="utf-8"?>
 <!DOCTYPE eagle SYSTEM "eagle.dtd">
-<eagle version="8.2.2">
+<eagle version="9.2.2">
 <drawing>
 <settings>
 <setting alwaysvectorfont="yes"/>
+<setting keepoldvectorfont="yes"/>
 <setting verticaltext="up"/>
 </settings>
@@
 <param name="dpMaxLengthDifference" value="10mm"/>
 <param name="dpGapFactor" value="2.5"/>
-<param name="checkGrid" value="0"/>
 <param name="checkAngle" value="0"/>
 <param name="checkFont" value="1"/>
 <param name="checkRestrict" value="1"/>
+<param name="checkStop" value="0"/>
+<param name="checkValues" value="0"/>
+<param name="checkNames" value="1"/>
+<param name="checkWireStubs" value="1"/>
+<param name="checkPolygonWidth" value="0"/>
 <param name="useDiameter" value="13"/>
 <param name="maxErrors" value="50"/>
@@
 </autorouter>
 <elements>
-<element name="C1" library="SparkFun-Capacitors" package="0603" value="0.1uF" x="26" y="40.4" rot="R180">
+<element name="C1" library="SparkFun-Capacitors" package="0603" value="0.1uF" x="26" y="40.4" smashed="yes" rot="R180">
+<attribute name="NAME" x="26" y="39.638" size="0.6096" layer="25" font="vector" ratio="20" rot="R180" align="bottom-center"/>
 <attribute name="PROD_ID" value="CAP-00810" x="26" y="40.4" size="1.778" layer="27" rot="R180" display="off"/>
-</element>
-<element name="C2" library="SparkFun-Capacitors" package="0603" value="0.1uF" x="43.5" y="35.5" rot="R180">
+<attribute name="VALUE" x="26" y="41.162" size="0.6096" layer="27" font="vector" ratio="20" rot="R180" align="top-center"/>
+</element>
+<element name="C2" library="SparkFun-Capacitors" package="0603" value="0.1uF" x="43.5" y="35.5" smashed="yes" rot="R180">
+<attribute name="NAME" x="43.5" y="34.738" size="0.6096" layer="25" font="vector" ratio="20" rot="R180" align="bottom-center"/>
 <attribute name="PROD_ID" value="CAP-00810" x="43.5" y="35.5" size="1.778" layer="27" rot="R180" display="off"/>
-</element>
-<element name="J1" library="WM6787CT-ND" package="WM6787CT-ND" value="WM6787CT-ND" x="37" y="25" rot="R90"/>
-<element name="J2" library="SparkFun-Connectors" package="1X02" value="" x="11.64" y="4.8"/>
-<element name="J3" library="SparkFun-Connectors" package="1X01" value="" x="31.4" y="4.8"/>
-<element name="Q1" library="SparkFun-DiscreteSemi" package="SOT23-3" value="BSS138" x="38.2" y="38.2" rot="R270">
+<attribute name="VALUE" x="43.5" y="36.262" size="0.6096" layer="27" font="vector" ratio="20" rot="R180" align="top-center"/>
+</element>
+<element name="J1" library="WM6787CT-ND" package="WM6787CT-ND" value="WM6787CT-ND" x="37" y="25" smashed="yes" rot="R90">
+<attribute name="NAME" x="35.8316" y="33.509" size="0.4064" layer="25"/>
+<attribute name="VALUE" x="35.349" y="32.493" size="0.6096" layer="27"/>
+</element>
+<element name="J2" library="SparkFun-Connectors" package="1X02" value="" x="11.64" y="4.8" smashed="yes">
+<attribute name="NAME" x="10.37" y="6.197" size="0.6096" layer="25" font="vector" ratio="20"/>
+<attribute name="VALUE" x="10.37" y="2.768" size="0.6096" layer="27" font="vector" ratio="20"/>
+</element>
+<element name="J3" library="SparkFun-Connectors" package="1X01" value="" x="31.4" y="4.8" smashed="yes">
+<attribute name="NAME" x="30.13" y="6.197" size="0.6096" layer="25" font="vector" ratio="20"/>
+<attribute name="VALUE" x="30.13" y="3.276" size="0.6096" layer="27" font="vector" ratio="20" align="top-left"/>
+</element>
+<element name="Q1" library="SparkFun-DiscreteSemi" package="SOT23-3" value="BSS138" x="38.2" y="38.2" smashed="yes" rot="R270">
+<attribute name="NAME" x="38.2" y="39.851" size="0.6096" layer="25" font="vector" ratio="20" align="bottom-center"/>
 <attribute name="PROD_ID" value="TRANS-00830" x="38.2" y="38.2" size="1.778" layer="27" rot="R270" display="off"/>
-</element>
-<element name="Q2" library="SparkFun-DiscreteSemi" package="SOT23-3" value="BSS138" x="38.1" y="43.3" rot="R270">
+<attribute name="VALUE" x="38.2" y="36.549" size="0.6096" layer="27" font="vector" ratio="20" align="top-center"/>
+</element>
+<element name="Q2" library="SparkFun-DiscreteSemi" package="SOT23-3" value="BSS138" x="38.1" y="43.3" smashed="yes" rot="R270">
+<attribute name="NAME" x="38.1" y="44.951" size="0.6096" layer="25" font="vector" ratio="20" align="bottom-center"/>
 <attribute name="PROD_ID" value="TRANS-00830" x="38.1" y="43.3" size="1.778" layer="27" rot="R270" display="off"/>
-</element>
-<element name="R1" library="SparkFun-Resistors" package="0603" value="10k" x="34.3" y="38.25" rot="R90">
+<attribute name="VALUE" x="38.1" y="41.649" size="0.6096" layer="27" font="vector" ratio="20" align="top-center"/>
+</element>
+<element name="R1" library="SparkFun-Resistors" package="0603" value="10k" x="34.3" y="38.25" smashed="yes" rot="R90">
+<attribute name="NAME" x="33.538" y="38.25" size="0.6096" layer="25" font="vector" ratio="20" rot="R90" align="bottom-center"/>
 <attribute name="PROD_ID" value="RES-00824" x="34.3" y="38.25" size="1.778" layer="27" rot="R90" display="off"/>
-</element>
-<element name="R2" library="SparkFun-Resistors" package="0603" value="10k" x="42.4" y="39" rot="R90">
+<attribute name="VALUE" x="35.062" y="38.25" size="0.6096" layer="27" font="vector" ratio="20" rot="R90" align="top-center"/>
+</element>
+<element name="R2" library="SparkFun-Resistors" package="0603" value="10k" x="42.4" y="39" smashed="yes" rot="R90">
+<attribute name="NAME" x="41.638" y="39" size="0.6096" layer="25" font="vector" ratio="20" rot="R90" align="bottom-center"/>
 <attribute name="PROD_ID" value="RES-00824" x="42.4" y="39" size="1.778" layer="27" rot="R90" display="off"/>
-</element>
-<element name="R3" library="SparkFun-Resistors" package="0603" value="10k" x="42.3" y="44.2" rot="R90">
+<attribute name="VALUE" x="43.162" y="39" size="0.6096" layer="27" font="vector" ratio="20" rot="R90" align="top-center"/>
+</element>
+<element name="R3" library="SparkFun-Resistors" package="0603" value="10k" x="42.3" y="44.2" smashed="yes" rot="R90">
+<attribute name="NAME" x="41.538" y="44.2" size="0.6096" layer="25" font="vector" ratio="20" rot="R90" align="bottom-center"/>
 <attribute name="PROD_ID" value="RES-00824" x="42.3" y="44.2" size="1.778" layer="27" rot="R90" display="off"/>
-</element>
-<element name="R4" library="SparkFun-Resistors" package="0603" value="10k" x="34.3" y="43.35" rot="R90">
+<attribute name="VALUE" x="43.062" y="44.2" size="0.6096" layer="27" font="vector" ratio="20" rot="R90" align="top-center"/>
+</element>
+<element name="R4" library="SparkFun-Resistors" package="0603" value="10k" x="34.3" y="43.35" smashed="yes" rot="R90">
+<attribute name="NAME" x="33.538" y="43.35" size="0.6096" layer="25" font="vector" ratio="20" rot="R90" align="bottom-center"/>
 <attribute name="PROD_ID" value="RES-00824" x="34.3" y="43.35" size="1.778" layer="27" rot="R90" display="off"/>
-</element>
-<element name="R5" library="SparkFun-Resistors" package="0603" value="715" x="18.1" y="4.8">
+<attribute name="VALUE" x="35.062" y="43.35" size="0.6096" layer="27" font="vector" ratio="20" rot="R90" align="top-center"/>
+</element>
+<element name="R5" library="SparkFun-Resistors" package="0603" value="715" x="18.1" y="4.8" smashed="yes">
+<attribute name="NAME" x="18.1" y="5.562" size="0.6096" layer="25" font="vector" ratio="20" align="bottom-center"/>
 <attribute name="PROD_ID" value="RES-07850" x="18.1" y="4.8" size="1.778" layer="27" display="off"/>
-</element>
-<element name="U1" library="Teensy_LC" package="TEENSY_LC" value="TEENSY_LC" x="11.66" y="25.05" rot="R270"/>
-<element name="U2" library="TLV810SDBZT" package="SOT95P237X112-3N" value="TLV810SDBZT" x="44.6" y="31.9">
+<attribute name="VALUE" x="18.1" y="4.038" size="0.6096" layer="27" font="vector" ratio="20" align="top-center"/>
+</element>
+<element name="U1" library="Teensy_LC" package="TEENSY_LC" value="TEENSY_LC" x="11.66" y="25.05" smashed="yes" rot="R270"/>
+<element name="U2" library="TLV810SDBZT" package="SOT95P237X112-3N" value="TLV810SDBZT" x="44.6" y="31.9" smashed="yes">
 <attribute name="AVAILABILITY" value="Unavailable" x="44.6" y="31.9" size="1.778" layer="27" display="off"/>
 <attribute name="DESCRIPTION" value=" 3-Pin Voltage Supervisors with Active-High, Push-Pull Reset 3-SOT-23 -40 to 125 " x="44.6" y="31.9" size="1.778" layer="27" display="off"/>
 <attribute name="MF" value="Texas Instruments" x="44.6" y="31.9" size="1.778" layer="27" display="off"/>
 <attribute name="MP" value="TLV810SDBZT" x="44.6" y="31.9" size="1.778" layer="27" display="off"/>
+<attribute name="NAME" x="44.065859375" y="33.678540625" size="0.6096" layer="25" ratio="10" rot="SR0"/>
 <attribute name="PACKAGE" value="TO-236 Texas Instruments" x="44.6" y="31.9" size="1.778" layer="27" display="off"/>
 <attribute name="PRICE" value="None" x="44.6" y="31.9" size="1.778" layer="27" display="off"/>
 </element>
+<element name="U$1" library="oshw" package="OSHW_5MM" value="" x="39.8" y="6.2" smashed="yes"/>
 </elements>
 <signals>
@@
 </signal>
 </signals>
+<mfgpreviewcolors>
+<mfgpreviewcolor name="soldermaskcolor" color="0xC8008000"/>
+<mfgpreviewcolor name="silkscreencolor" color="0xFFFEFEFE"/>
+<mfgpreviewcolor name="backgroundcolor" color="0xFF282828"/>
+<mfgpreviewcolor name="coppercolor" color="0xFFFFBF00"/>
+<mfgpreviewcolor name="substratecolor" color="0xFF786E46"/>
+</mfgpreviewcolors>
 </board>
 </drawing>
+<compatibility>
+<note version="6.3" minversion="6.2.2" severity="warning">
+Since Version 6.2.2 text objects can contain more than one line,
+which will not be processed correctly with this version.
+</note>
+</compatibility>
 </eagle>

Commit message: Add files via upload
Parts:
- added GOLD_ORB_SM1: OSHWLOGOLOGO5MM, oshw:OSHW_5MM
- J2: value (none) -> 2
- J3: value (none) -> 3
- Q1, Q2: value BSS138 -> 220mA/50V/3.5Ω
Changed lines of the file:
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@@
 <layers>
 <layer number="1" name="Top" color="4" fill="1" visible="yes" active="yes"/>
+<layer number="2" name="Route2" color="1" fill="3" visible="yes" active="yes"/>
+<layer number="15" name="Route15" color="4" fill="6" visible="yes" active="yes"/>
 <layer number="16" name="Bottom" color="1" fill="1" visible="yes" active="yes"/>
 <layer number="17" name="Pads" color="2" fill="1" visible="yes" active="yes"/>
@@
 <attribute name="VALUE" x="35.349" y="32.493" size="0.6096" layer="27"/>
 </element>
-<element name="J2" library="SparkFun-Connectors" package="1X02" value="" x="11.64" y="4.8" smashed="yes">
+<element name="J2" library="SparkFun-Connectors" package="1X02" value="2" x="11.64" y="4.8" smashed="yes">
 <attribute name="NAME" x="10.37" y="6.197" size="0.6096" layer="25" font="vector" ratio="20"/>
 <attribute name="VALUE" x="10.37" y="2.768" size="0.6096" layer="27" font="vector" ratio="20"/>
 </element>
-<element name="J3" library="SparkFun-Connectors" package="1X01" value="" x="31.4" y="4.8" smashed="yes">
+<element name="J3" library="SparkFun-Connectors" package="1X01" value="3" x="31.4" y="4.8" smashed="yes">
 <attribute name="NAME" x="30.13" y="6.197" size="0.6096" layer="25" font="vector" ratio="20"/>
 <attribute name="VALUE" x="30.13" y="3.276" size="0.6096" layer="27" font="vector" ratio="20" align="top-left"/>
 </element>
-<element name="Q1" library="SparkFun-DiscreteSemi" package="SOT23-3" value="BSS138" x="38.2" y="38.2" smashed="yes" rot="R270">
+<element name="Q1" library="SparkFun-DiscreteSemi" library_urn="urn:adsk.eagle:library:514" package="SOT23-3" package3d_urn="urn:adsk.eagle:package:38446/1" value="220mA/50V/3.5Ω" x="38.2" y="38.2" smashed="yes" rot="R270">
 <attribute name="NAME" x="38.2" y="39.851" size="0.6096" layer="25" font="vector" ratio="20" align="bottom-center"/>
 <attribute name="PROD_ID" value="TRANS-00830" x="38.2" y="38.2" size="1.778" layer="27" rot="R270" display="off"/>
 <attribute name="VALUE" x="38.2" y="36.549" size="0.6096" layer="27" font="vector" ratio="20" align="top-center"/>
 </element>
-<element name="Q2" library="SparkFun-DiscreteSemi" package="SOT23-3" value="BSS138" x="38.1" y="43.3" smashed="yes" rot="R270">
+<element name="Q2" library="SparkFun-DiscreteSemi" library_urn="urn:adsk.eagle:library:514" package="SOT23-3" package3d_urn="urn:adsk.eagle:package:38446/1" value="220mA/50V/3.5Ω" x="38.1" y="43.3" smashed="yes" rot="R270">
 <attribute name="NAME" x="38.1" y="44.951" size="0.6096" layer="25" font="vector" ratio="20" align="bottom-center"/>
 <attribute name="PROD_ID" value="TRANS-00830" x="38.1" y="43.3" size="1.778" layer="27" rot="R270" display="off"/>
@@
 </element>
 <element name="U$1" library="oshw" package="OSHW_5MM" value="" x="39.8" y="6.2" smashed="yes"/>
+<element name="GOLD_ORB_SM1" library="oshw" package="OSHW_5MM" value="OSHWLOGOLOGO5MM" x="4.9" y="-2.5" smashed="yes"/>
 </elements>
 <signals>
@@
 which will not be processed correctly with this version.
 </note>
+<note version="8.2" severity="warning">
+Since Version 8.2, EAGLE supports online libraries. The ids
+of those online libraries will not be understood (or retained)
+with this version.
+</note>
+<note version="8.3" severity="warning">
+Since Version 8.3, EAGLE supports URNs for individual library
+assets (packages, symbols, and devices). The URNs of those assets
+will not be understood (or retained) with this version.
+</note>
+<note version="8.3" severity="warning">
+Since Version 8.3, EAGLE supports the association of 3D packages
+with devices in libraries, schematics, and board files. Those 3D
+packages will not be understood (or retained) with this version.
+</note>
 </compatibility>
