File: Example_Keyboards/Lenovo_ThinkPad_T61/Teensy LC/Eagle/T61_LC_Scanner.sch (EAGLE design)
At the start: 14 parts, among them J1 WM6787CT-ND, Q1 BSS138, Q2 BSS138, U1 TEENSY_LC, U2 TLV810SDBZT

Commit message: Add files via upload
Changed lines of the file:
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@@
 <?xml version="1.0" encoding="utf-8"?>
 <!DOCTYPE eagle SYSTEM "eagle.dtd">
-<eagle version="8.2.2">
+<eagle version="9.2.2">
 <drawing>
 <settings>
 <setting alwaysvectorfont="yes"/>
+<setting keepoldvectorfont="yes"/>
 <setting verticaltext="up"/>
 </settings>
@@
 <text x="101.092" y="-1.778" size="1.778" layer="91">5V</text>
 <text x="17.526" y="30.988" size="1.778" layer="91">5V</text>
-<text x="-41.148" y="44.45" size="1.778" layer="91">NO CONNECTS</text>
+<text x="-46.228" y="44.45" size="1.778" layer="91">NO CONNECTS</text>
 <text x="16.764" y="97.028" size="1.778" layer="91">SENSE(0)</text>
 <text x="16.764" y="94.234" size="1.778" layer="91">SENSE(1)</text>
@@
 </plain>
 <instances>
-<instance part="U1" gate="G$1" x="0" y="63.5"/>
-<instance part="J1" gate="G$1" x="157.48" y="71.12"/>
-<instance part="U2" gate="A" x="81.28" y="17.78"/>
-<instance part="Q1" gate="NMOS" x="81.28" y="-15.24" rot="R270"/>
-<instance part="Q2" gate="NMOS" x="81.28" y="-33.02" rot="R270"/>
-<instance part="R1" gate="G$1" x="71.12" y="-10.16" rot="R90"/>
-<instance part="R2" gate="G$1" x="91.44" y="-10.16" rot="R90"/>
-<instance part="R3" gate="G$1" x="96.52" y="-27.94" rot="R90"/>
-<instance part="R4" gate="G$1" x="66.04" y="-27.94" rot="R90"/>
-<instance part="R5" gate="G$1" x="-33.02" y="5.08"/>
-<instance part="J2" gate="G$1" x="-55.88" y="2.54"/>
-<instance part="J3" gate="G$1" x="185.42" y="53.34" rot="R180"/>
-<instance part="C1" gate="G$1" x="40.64" y="-10.16"/>
-<instance part="C2" gate="G$1" x="58.42" y="12.7"/>
+<instance part="U1" gate="G$1" x="0" y="63.5" smashed="yes">
+<attribute name="NAME" x="-5.08" y="101.6" size="1.778" layer="94"/>
+<attribute name="VALUE" x="-5.08" y="-17.78" size="1.778" layer="94"/>
+</instance>
+<instance part="J1" gate="G$1" x="157.48" y="71.12" smashed="yes">
+<attribute name="NAME" x="160.02" y="114.3" size="1.778" layer="95" rot="MR0"/>
+<attribute name="VALUE" x="152.4" y="-50.8" size="1.778" layer="96"/>
+</instance>
+<instance part="U2" gate="A" x="81.28" y="17.78" smashed="yes">
+<attribute name="NAME" x="75.91195" y="26.91331875" size="2.086159375" layer="95" ratio="10" rot="SR0"/>
+</instance>
+<instance part="Q1" gate="NMOS" x="81.28" y="-15.24" smashed="yes" rot="R270">
+<attribute name="NAME" x="81.28" y="-20.32" size="1.778" layer="95" font="vector" rot="R270"/>
+<attribute name="VALUE" x="78.74" y="-20.32" size="1.778" layer="96" font="vector" rot="R270"/>
+</instance>
+<instance part="Q2" gate="NMOS" x="81.28" y="-33.02" smashed="yes" rot="R270">
+<attribute name="NAME" x="81.28" y="-38.1" size="1.778" layer="95" font="vector" rot="R270"/>
+<attribute name="VALUE" x="78.74" y="-38.1" size="1.778" layer="96" font="vector" rot="R270"/>
+</instance>
+<instance part="R1" gate="G$1" x="71.12" y="-10.16" smashed="yes" rot="R90">
+<attribute name="NAME" x="69.596" y="-10.16" size="1.778" layer="95" font="vector" rot="R90" align="bottom-center"/>
+<attribute name="VALUE" x="72.644" y="-10.16" size="1.778" layer="96" font="vector" rot="R90" align="top-center"/>
+</instance>
+<instance part="R2" gate="G$1" x="91.44" y="-10.16" smashed="yes" rot="R90">
+<attribute name="NAME" x="89.916" y="-10.16" size="1.778" layer="95" font="vector" rot="R90" align="bottom-center"/>
+<attribute name="VALUE" x="92.964" y="-10.16" size="1.778" layer="96" font="vector" rot="R90" align="top-center"/>
+</instance>
+<instance part="R3" gate="G$1" x="96.52" y="-27.94" smashed="yes" rot="R90">
+<attribute name="NAME" x="94.996" y="-27.94" size="1.778" layer="95" font="vector" rot="R90" align="bottom-center"/>
+<attribute name="VALUE" x="98.044" y="-27.94" size="1.778" layer="96" font="vector" rot="R90" align="top-center"/>
+</instance>
+<instance part="R4" gate="G$1" x="66.04" y="-27.94" smashed="yes" rot="R90">
+<attribute name="NAME" x="64.516" y="-27.94" size="1.778" layer="95" font="vector" rot="R90" align="bottom-center"/>
+<attribute name="VALUE" x="67.564" y="-27.94" size="1.778" layer="96" font="vector" rot="R90" align="top-center"/>
+</instance>
+<instance part="R5" gate="G$1" x="-33.02" y="5.08" smashed="yes">
+<attribute name="NAME" x="-33.02" y="6.604" size="1.778" layer="95" font="vector" align="bottom-center"/>
+<attribute name="VALUE" x="-33.02" y="3.556" size="1.778" layer="96" font="vector" align="top-center"/>
+</instance>
+<instance part="J2" gate="G$1" x="-55.88" y="2.54" smashed="yes">
+<attribute name="VALUE" x="-58.42" y="-2.286" size="1.778" layer="96" font="vector"/>
+<attribute name="NAME" x="-58.42" y="8.128" size="1.778" layer="95" font="vector"/>
+</instance>
+<instance part="J3" gate="G$1" x="185.42" y="53.34" smashed="yes" rot="R180">
+<attribute name="VALUE" x="187.96" y="58.166" size="1.778" layer="96" font="vector" rot="R180"/>
+<attribute name="NAME" x="187.96" y="50.292" size="1.778" layer="95" font="vector" rot="R180"/>
+</instance>
+<instance part="C1" gate="G$1" x="40.64" y="-10.16" smashed="yes">
+<attribute name="NAME" x="42.164" y="-7.239" size="1.778" layer="95" font="vector"/>
+<attribute name="VALUE" x="42.164" y="-12.319" size="1.778" layer="96" font="vector"/>
+</instance>
+<instance part="C2" gate="G$1" x="58.42" y="12.7" smashed="yes">
+<attribute name="NAME" x="59.944" y="15.621" size="1.778" layer="95" font="vector"/>
+<attribute name="VALUE" x="59.944" y="10.541" size="1.778" layer="96" font="vector"/>
+</instance>
 </instances>
 <busses>

Commit message: Add files via upload
Parts:
- added GOLD_ORB_SM1: OSHWLOGOLOGO5MM, oshw:OSHWLOGOLOGO5MM
- J2: value (none) -> 2
- J3: value (none) -> 3
- Q1, Q2: value BSS138 -> 220mA/50V/3.5Ω
Changed lines of the file:
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@@
 <layers>
 <layer number="1" name="Top" color="4" fill="1" visible="no" active="no"/>
+<layer number="2" name="Route2" color="1" fill="3" visible="no" active="no"/>
+<layer number="15" name="Route15" color="4" fill="6" visible="no" active="no"/>
 <layer number="16" name="Bottom" color="1" fill="1" visible="no" active="no"/>
 <layer number="17" name="Pads" color="2" fill="1" visible="no" active="no"/>
@@
 <part name="J1" library="WM6787CT-ND" deviceset="WM6787CT-ND" device="" value="WM6787CT-ND"/>
 <part name="U2" library="TLV810SDBZT" deviceset="TLV810SDBZT" device=""/>
-<part name="Q1" library="SparkFun-DiscreteSemi" deviceset="MOSFET-NCH" device="-BSS138" value="BSS138"/>
-<part name="Q2" library="SparkFun-DiscreteSemi" deviceset="MOSFET-NCH" device="-BSS138" value="BSS138"/>
+<part name="Q1" library="SparkFun-DiscreteSemi" library_urn="urn:adsk.eagle:library:514" deviceset="MOSFET-NCH" device="-BSS138" package3d_urn="urn:adsk.eagle:package:38446/1" value="220mA/50V/3.5Ω"/>
+<part name="Q2" library="SparkFun-DiscreteSemi" library_urn="urn:adsk.eagle:library:514" deviceset="MOSFET-NCH" device="-BSS138" package3d_urn="urn:adsk.eagle:package:38446/1" value="220mA/50V/3.5Ω"/>
 <part name="R1" library="SparkFun-Resistors" deviceset="10KOHM" device="-0603-1/10W-1%" value="10k"/>
 <part name="R2" library="SparkFun-Resistors" deviceset="10KOHM" device="-0603-1/10W-1%" value="10k"/>
@@
 <part name="R4" library="SparkFun-Resistors" deviceset="10KOHM" device="-0603-1/10W-1%" value="10k"/>
 <part name="R5" library="SparkFun-Resistors" deviceset="715OHM" device="-0603-1/10W-1%" value="715"/>
-<part name="J2" library="SparkFun-Connectors" deviceset="CONN_02" device=""/>
-<part name="J3" library="SparkFun-Connectors" deviceset="CONN_01" device=""/>
+<part name="J2" library="SparkFun-Connectors" deviceset="CONN_02" device="" value="2"/>
+<part name="J3" library="SparkFun-Connectors" deviceset="CONN_01" device="" value="3"/>
 <part name="C1" library="SparkFun-Capacitors" deviceset="0.1UF" device="-0603-25V-(+80/-20%)" value="0.1uF"/>
 <part name="C2" library="SparkFun-Capacitors" deviceset="0.1UF" device="-0603-25V-(+80/-20%)" value="0.1uF"/>
+<part name="GOLD_ORB_SM1" library="oshw" deviceset="OSHWLOGO" device="LOGO5MM"/>
 </parts>
 <sheets>
@@
 <attribute name="VALUE" x="59.944" y="10.541" size="1.778" layer="96" font="vector"/>
 </instance>
+<instance part="GOLD_ORB_SM1" gate="G$1" x="-12.7" y="-45.72" smashed="yes"/>
 </instances>
 <busses>
@@
 </schematic>
 </drawing>
+<compatibility>
+<note version="6.3" minversion="6.2.2" severity="warning">
+Since Version 6.2.2 text objects can contain more than one line,
+which will not be processed correctly with this version.
+</note>
+<note version="8.2" severity="warning">
+Since Version 8.2, EAGLE supports online libraries. The ids
+of those online libraries will not be understood (or retained)
+with this version.
+</note>
+<note version="8.3" severity="warning">
+Since Version 8.3, EAGLE supports URNs for individual library
+assets (packages, symbols, and devices). The URNs of those assets
+will not be understood (or retained) with this version.
+</note>
+<note version="8.3" severity="warning">
+Since Version 8.3, EAGLE supports the association of 3D packages
+with devices in libraries, schematics, and board files. Those 3D
+packages will not be understood (or retained) with this version.
+</note>
+</compatibility>
 </eagle>
