File: IBM T43 Files/T43.kicad_pcb (KiCad board)
At the start: 2 copper layers, 49.8 x 49.8 mm, 14 parts

Commit message: Add files via upload
Parts:
- added ?: , , F.Cu at (108.1, 82.5)
- added ?: , , F.Cu at (139.8, 97.2)
Other:
- board text added: "24"
- board text added: "25"
- board text added: "26"
- board text added: "31"
- board text added: "32"
- board text added: "33"
- board text added: "Blink"
- board text added: "Cap"
- board text added: "IBM T43 Controller"
- board text added: "JAE KX14-40K5DE"
- board text added: "Num"
- board text added: "Scrl"
- board text added: "Sync"
- board text added: "Version 1.2"
- board text removed: "Lenovo T43 Controller"
- board text removed: "Version 1.1"

Commit message: Add files via upload
Changed lines of the file:
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@@
       (effects (font (size 1.27 1.27) (thickness 0.15)))
-    )
-    (fp_text user KX14-40K5DE (at 139.75 94.95 -180) (layer F.SilkS)
-      (effects (font (size 1 1) (thickness 0.15)))
     )
   )
@@
       (effects (font (size 1.27 1.27) (thickness 0.15)))
     )
-    (fp_text user KX14-40K5DE (at 135.175 85.65 -180) (layer F.SilkS)
-      (effects (font (size 1 1) (thickness 0.15)))
-    )
   )
