File: Keyboard_Scanner_Eagle_Layouts/Keyboard_Scanner_LC_thruhole.brd (EAGLE design)
At the start: 37 x 69 mm, 3 parts, among them J1 1.00MM DIP FPC

Commit message: Add files via upload
Parts:
- moved U$2 21.6 mm to (27.0, 43.5)
- moved U$1 10.0 mm to (12.7, 24.1)
- moved J1 2.50 mm to (32.4, 11.6)
Routing:
- net IO_0: track 13.8 -> 11.0 mm
- net IO_22: track 33.3 -> 30.7 mm
- net IO_1: track 13.2 -> 10.8 mm
- net IO_24: track 29.1 -> 26.9 mm
- net IO_23: track 33.9 -> 31.8 mm
- net IO_2: track 12.6 -> 10.6 mm
- net IO_12: track 13.5 -> 11.7 mm
- net IO_21: track 31.1 -> 29.3 mm
- net IO_3: track 11.9 -> 10.3 mm
- net IO_11: track 12.9 -> 11.5 mm
- net IO_25: track 26.9 -> 25.5 mm
- net IO_26: track 28.3 -> 27.0 mm
- net IO_10: track 12.5 -> 11.2 mm
- net IO_4: track 11.3 -> 10.1 mm
- net IO_15: track 30.1 -> 29.0 mm
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Other:
- board size 37 x 69 mm -> 37 x 48 mm
