File: Keyboard_Scanner_Eagle_Layouts/FPC_10pin0p5mm.brd (EAGLE design)
At the start: 17 x 17 mm, 2 parts

Commit message: Add files via upload
Parts:
- added J3: J3, SparkFun-Connectors:1X01
- added J4: J4, SparkFun-Connectors:1X01
- added J5: J5, SparkFun-Connectors:1X01
- added Q1: MMBF170, MMBF170:MMBF170
- added R1: 1206, R1206:R1206
- J1: value (none) -> J1
- J2: value (none) -> J2
- moved J1 1.00 mm to (10.5, 5.48)
- moved J2 1.00 mm to (4.58, 2.04)
Connections:
- new net N$11: Q1.3, R1.1
- new net N$12: J3.1, R1.2
- new net N$13: J4.1, Q1.1
- net GND: now also J5.1, Q1.2
Routing:
- net N$12: track 0.00 -> 15.5 mm
- net N$13: track 0.00 -> 10.4 mm
- net GND: track 9.42 -> 0.00 mm, vias 1 -> 0
- net N$11: track 0.00 -> 5.03 mm
- net N$4: track 7.80 -> 8.76 mm
- net N$2: track 8.44 -> 9.40 mm
- net N$3: track 5.05 -> 6.02 mm
- net N$5: track 4.45 -> 5.40 mm
- net N$1: track 5.74 -> 6.67 mm
- net N$6: track 7.79 -> 8.47 mm
- net N$8: track 8.43 -> 9.08 mm
- net N$9: track 5.72 -> 6.36 mm
- net N$7: track 5.08 -> 5.72 mm
Other:
- board text added: "0.5mm pitch"
- board text added: "1"
- board text added: "1206"
- board text added: "D"
- board text added: "Drain"
- board text added: "G"
- board text added: "GND"
- board text added: "Gate"
- board text added: "MMBF170"
- board text added: "S"
- board text removed: "10pin0.5mm"
