File: Example_Keyboards/Pico_T61_Keyboard/Eagle_Layout/Pico_T61_Keyboard.sch (EAGLE design)
At the start: 20 parts, among them IC1 TPS60150DRVR, IC2 TLV810MDBZR, J2 JST-PH-3PIN, J4 JST-PH-2PIN, J5 AA01B-S040, Q1 220mA/50V/3.5Ω, Q2 220mA/50V/3.5Ω, U1 SC0918

Commit message: Add files via upload
Parts:
- J1, J3: device SparkFun-Connectors:CONN_01PTH_NO_SILK_KIT -> SparkFun-Connectors:CONN_01
Changed lines of the file:
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@@
 <part name="C3" library="0603_CAP" deviceset="0603_CAP" device="" value="2.2UF"/>
 <part name="R1" library="SparkFun-Resistors" library_urn="urn:adsk.eagle:library:532" deviceset="10KOHM" device="-0603-1/10W-1%" package3d_urn="urn:adsk.eagle:package:39650/1" value="10k"/>
-<part name="J3" library="SparkFun-Connectors" library_urn="urn:adsk.eagle:library:513" deviceset="CONN_01" device="PTH_NO_SILK_KIT" package3d_urn="urn:adsk.eagle:package:38038/1"/>
-<part name="J1" library="SparkFun-Connectors" library_urn="urn:adsk.eagle:library:513" deviceset="CONN_01" device="PTH_NO_SILK_KIT" package3d_urn="urn:adsk.eagle:package:38038/1"/>
+<part name="J3" library="SparkFun-Connectors" library_urn="urn:adsk.eagle:library:513" deviceset="CONN_01" device="" package3d_urn="urn:adsk.eagle:package:38028/1"/>
+<part name="J1" library="SparkFun-Connectors" library_urn="urn:adsk.eagle:library:513" deviceset="CONN_01" device="" package3d_urn="urn:adsk.eagle:package:38028/1"/>
 <part name="J2" library="JST-PH-3PIN" deviceset="JST-PH-3PIN" device="" value="JST-PH-3PIN"/>
 </parts>
