File: Example_Keyboards/Pico_T61_Keyboard/Eagle_Layout/Pico_T61_Keyboard.brd (EAGLE design)
At the start: 55 x 55 mm, 22 parts, among them IC1 TPS60150DRVR, IC2 TLV810MDBZR, J2 JST-PH-3PIN, J4 JST-PH-2PIN, J5 AA01B-S040, Q1 220mA/50V/3.5Ω, Q2 220mA/50V/3.5Ω, U1 SC0918

Commit message: Add files via upload
Parts:
- J1, J3: device SparkFun-Connectors:1X01NS_KIT -> SparkFun-Connectors:1X01
Changed lines of the file:
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@@
 <text x="48.4" y="40.6" size="0.6096" layer="21" ratio="15" rot="R180">C3</text>
 <text x="53.7" y="38.8" size="0.6096" layer="21" ratio="15" rot="R270">C4</text>
-<text x="51" y="30.7" size="0.6096" layer="21" ratio="15">TP PWR</text>
-<text x="29.4" y="52.7" size="0.6096" layer="21" ratio="15">USB PWR</text>
+<text x="51.2" y="30.4" size="0.6096" layer="21" ratio="15">TP PWR</text>
+<text x="29" y="53.5" size="0.6096" layer="21" ratio="15">USB PWR</text>
 <wire x1="36.4" y1="42.9" x2="36.4" y2="44.2" width="0.1524" layer="21"/>
 <wire x1="36.4" y1="44.2" x2="39.6" y2="44.2" width="0.1524" layer="21"/>
@@
 <attribute name="VALUE" x="50.762" y="46.7" size="0.6096" layer="27" font="vector" ratio="20" rot="R90" align="top-center"/>
 </element>
-<element name="J3" library="SparkFun-Connectors" library_urn="urn:adsk.eagle:library:513" package="1X01NS_KIT" package3d_urn="urn:adsk.eagle:package:38038/1" value="" x="52.7" y="32.5" smashed="yes">
-<attribute name="NAME" x="51.43" y="33.643" size="0.6096" layer="25" font="vector" ratio="20"/>
+<element name="J3" library="SparkFun-Connectors" library_urn="urn:adsk.eagle:library:513" package="1X01" package3d_urn="urn:adsk.eagle:package:38028/1" value="" x="52.7" y="32.5" smashed="yes">
+<attribute name="NAME" x="52.23" y="34.043" size="0.6096" layer="25" font="vector" ratio="20"/>
 <attribute name="VALUE" x="51.43" y="31.484" size="0.6096" layer="27" font="vector" ratio="20" align="top-left"/>
 </element>
-<element name="J1" library="SparkFun-Connectors" library_urn="urn:adsk.eagle:library:513" package="1X01NS_KIT" package3d_urn="urn:adsk.eagle:package:38038/1" value="" x="34.1" y="52.7" smashed="yes">
-<attribute name="NAME" x="32.13" y="51.743" size="0.6096" layer="25" font="vector" ratio="20"/>
+<element name="J1" library="SparkFun-Connectors" library_urn="urn:adsk.eagle:library:513" package="1X01" package3d_urn="urn:adsk.eagle:package:38028/1" value="" x="34.1" y="52.7" smashed="yes">
+<attribute name="NAME" x="31.63" y="52.343" size="0.6096" layer="25" font="vector" ratio="20"/>
 <attribute name="VALUE" x="32.83" y="51.684" size="0.6096" layer="27" font="vector" ratio="20" align="top-left"/>
 </element>
