File: Example_Keyboards/Pico_T61_Keyboard/Eagle_Layout/Pico_T420_Keyboard_R1.brd (EAGLE design)
At the start: 55 x 55 mm, 22 parts, among them IC1 TPS60150DRVR, IC2 TLV810MDBZR, J2 JST-PH-3PIN, J4 JST-PH-2PIN, J5 AA01B-S040, Q1 220mA/50V/3.5Ω, Q2 220mA/50V/3.5Ω, U1 SC0918

Commit message: Add files via upload
Parts:
- added J6, J7: (no value), JST-PH-2PIN:JST-PH-2PIN
- moved U$2 20.0 mm to (19.5, 29.8)
- moved U$1 0.22 mm to (36.7, 19.1)
Connections:
- new net N$1: J6.P$2, U1.30
- new net N$4: J7.P$2, U1.37
- net GND: now also J6.P$1, J7.P$1
Routing:
- net N$4: track 0.00 -> 26.7 mm
- net N$1: track 0.00 -> 25.7 mm
- net 37: track 41.3 -> 39.6 mm
Other:
- board text added: "5V"
- board text added: "EN"
- board text added: "GND"
- board text added: "KBSW"
- board text added: "RUN"
- board text added: "VBAT"
