File: Example_Keyboards/Pico_T61_Keyboard/Eagle_Layout/Pico_T61_Keyboard_R1.sch (EAGLE design)
At the start: 20 parts, among them IC1 TPS60150DRVR, IC2 TLV810MDBZR, J2 JST-PH-3PIN, J4 JST-PH-2PIN, J5 AA01B-S040, Q1 220mA/50V/3.5Ω, Q2 220mA/50V/3.5Ω, U1 SC0918

Commit message: Add files via upload
Parts:
- added J6, J7: (no value), JST-PH-2PIN:JST-PH-2PIN
Connections:
- new net N$1: J6.P2, U1.RUN
- new net N$4: J7.P2, U1.3V3_EN
- net GND: now also J6.P1, J7.P1
Other:
- note added: "To Power Down Switch"
- note added: "To Reset push button"
Changed lines of the file:
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@@
 <part name="Q1" library="SparkFun-DiscreteSemi" library_urn="urn:adsk.eagle:library:514" deviceset="MOSFET-NCH" device="-BSS138" package3d_urn="urn:adsk.eagle:package:38446/1" value="220mA/50V/3.5Ω"/>
 <part name="Q2" library="SparkFun-DiscreteSemi" library_urn="urn:adsk.eagle:library:514" deviceset="MOSFET-NCH" device="-BSS138" package3d_urn="urn:adsk.eagle:package:38446/1" value="220mA/50V/3.5Ω"/>
-<part name="R2" library="SparkFun-Resistors" library_urn="urn:adsk.eagle:library:532" deviceset="10KOHM" device="-0603-1/10W-1%" package3d_urn="urn:adsk.eagle:package:39650/1" value="10k"/>
-<part name="R4" library="SparkFun-Resistors" library_urn="urn:adsk.eagle:library:532" deviceset="10KOHM" device="-0603-1/10W-1%" package3d_urn="urn:adsk.eagle:package:39650/1" value="10k"/>
-<part name="R5" library="SparkFun-Resistors" library_urn="urn:adsk.eagle:library:532" deviceset="10KOHM" device="-0603-1/10W-1%" package3d_urn="urn:adsk.eagle:package:39650/1" value="10k"/>
-<part name="R3" library="SparkFun-Resistors" library_urn="urn:adsk.eagle:library:532" deviceset="10KOHM" device="-0603-1/10W-1%" package3d_urn="urn:adsk.eagle:package:39650/1" value="10k"/>
+<part name="R2" library="SparkFun-Resistors" deviceset="10KOHM" device="-0603-1/10W-1%" package3d_urn="urn:adsk.eagle:package:39650/1" value="10k"/>
+<part name="R4" library="SparkFun-Resistors" deviceset="10KOHM" device="-0603-1/10W-1%" package3d_urn="urn:adsk.eagle:package:39650/1" value="10k"/>
+<part name="R5" library="SparkFun-Resistors" deviceset="10KOHM" device="-0603-1/10W-1%" package3d_urn="urn:adsk.eagle:package:39650/1" value="10k"/>
+<part name="R3" library="SparkFun-Resistors" deviceset="10KOHM" device="-0603-1/10W-1%" package3d_urn="urn:adsk.eagle:package:39650/1" value="10k"/>
 <part name="SUPPLY3" library="supply2" library_urn="urn:adsk.eagle:library:372" deviceset="GND" device=""/>
 <part name="SUPPLY6" library="supply2" library_urn="urn:adsk.eagle:library:372" deviceset="GND" device=""/>
@@
 <part name="C2" library="0603_CAP" deviceset="0603_CAP" device="" value="2.2UF"/>
 <part name="C3" library="0603_CAP" deviceset="0603_CAP" device="" value="2.2UF"/>
-<part name="R1" library="SparkFun-Resistors" library_urn="urn:adsk.eagle:library:532" deviceset="10KOHM" device="-0603-1/10W-1%" package3d_urn="urn:adsk.eagle:package:39650/1" value="10k"/>
-<part name="J3" library="SparkFun-Connectors" library_urn="urn:adsk.eagle:library:513" deviceset="CONN_01" device="" package3d_urn="urn:adsk.eagle:package:38028/1"/>
-<part name="J1" library="SparkFun-Connectors" library_urn="urn:adsk.eagle:library:513" deviceset="CONN_01" device="" package3d_urn="urn:adsk.eagle:package:38028/1"/>
+<part name="R1" library="SparkFun-Resistors" deviceset="10KOHM" device="-0603-1/10W-1%" package3d_urn="urn:adsk.eagle:package:39650/1" value="10k"/>
+<part name="J3" library="SparkFun-Connectors" deviceset="CONN_01" device="" package3d_urn="urn:adsk.eagle:package:38028/1"/>
+<part name="J1" library="SparkFun-Connectors" deviceset="CONN_01" device="" package3d_urn="urn:adsk.eagle:package:38028/1"/>
 <part name="J2" library="JST-PH-3PIN" deviceset="JST-PH-3PIN" device="" value="JST-PH-3PIN"/>
+<part name="J6" library="JST-PH-2PIN" deviceset="JST-PH-2PIN" device=""/>
+<part name="J7" library="JST-PH-2PIN" deviceset="JST-PH-2PIN" device=""/>
+<part name="SUPPLY4" library="supply2" library_urn="urn:adsk.eagle:library:372" deviceset="GND" device=""/>
+<part name="SUPPLY10" library="supply2" library_urn="urn:adsk.eagle:library:372" deviceset="GND" device=""/>
 </parts>
 <sheets>
@@
 <text x="10.16" y="137.16" size="1.778" layer="97">If not using Bluetooth, use the USB 5 volts to power the Trackpoint.
 Add Jumper wire from J1 to J3 and do not install IC1, C1, C2, C3, R1, D1, and J2.  </text>
+<text x="-88.9" y="91.44" size="1.778" layer="97">To Reset push button</text>
+<text x="-60.96" y="91.44" size="1.778" layer="97">To Power Down Switch</text>
 </plain>
 <instances>
@@
 <attribute name="NAME" x="15.24" y="104.14" size="1.27" layer="95" rot="R90"/>
 <attribute name="VALUE" x="0" y="111.76" size="1.778" layer="96"/>
+</instance>
+<instance part="J6" gate="G$1" x="-76.2" y="83.82" smashed="yes" rot="R90">
+<attribute name="NAME" x="-83.82" y="76.2" size="1.778" layer="95" rot="R90"/>
+<attribute name="VALUE" x="-66.04" y="76.2" size="1.778" layer="96" rot="R90"/>
+</instance>
+<instance part="J7" gate="G$1" x="-55.88" y="83.82" smashed="yes" rot="R90">
+<attribute name="NAME" x="-63.5" y="76.2" size="1.778" layer="95" rot="R90"/>
+<attribute name="VALUE" x="-45.72" y="76.2" size="1.778" layer="96" rot="R90"/>
+</instance>
+<instance part="SUPPLY4" gate="GND" x="-78.74" y="71.12" smashed="yes">
+<attribute name="VALUE" x="-80.645" y="67.945" size="1.778" layer="96"/>
+</instance>
+<instance part="SUPPLY10" gate="GND" x="-58.42" y="71.12" smashed="yes">
+<attribute name="VALUE" x="-60.325" y="67.945" size="1.778" layer="96"/>
 </instance>
 </instances>
@@
 <wire x1="5.08" y1="93.98" x2="5.08" y2="96.52" width="0.1524" layer="91"/>
 </segment>
+<segment>
+<pinref part="J6" gate="G$1" pin="P1"/>
+<pinref part="SUPPLY4" gate="GND" pin="GND"/>
+<wire x1="-78.74" y1="76.2" x2="-78.74" y2="73.66" width="0.1524" layer="91"/>
+</segment>
+<segment>
+<pinref part="J7" gate="G$1" pin="P1"/>
+<pinref part="SUPPLY10" gate="GND" pin="GND"/>
+<wire x1="-58.42" y1="76.2" x2="-58.42" y2="73.66" width="0.1524" layer="91"/>
+</segment>
 </net>
 <net name="5" class="0">
@@
 </segment>
 </net>
+<net name="N$1" class="0">
+<segment>
+<pinref part="J6" gate="G$1" pin="P2"/>
+<wire x1="-73.66" y1="76.2" x2="-73.66" y2="53.34" width="0.1524" layer="91"/>
+<pinref part="U1" gate="G$1" pin="RUN"/>
+<wire x1="-73.66" y1="53.34" x2="-48.26" y2="53.34" width="0.1524" layer="91"/>
+</segment>
+</net>
+<net name="N$4" class="0">
+<segment>
+<pinref part="J7" gate="G$1" pin="P2"/>
+<pinref part="U1" gate="G$1" pin="3V3_EN"/>
+<wire x1="-53.34" y1="76.2" x2="-53.34" y2="55.88" width="0.1524" layer="91"/>
+<wire x1="-53.34" y1="55.88" x2="-48.26" y2="55.88" width="0.1524" layer="91"/>
+</segment>
+</net>
