File: Example_Keyboards/Pico_26Pin_Keyboard/Pico_26Pin_Keyboard.brd (EAGLE design)
At the start: 55 x 55 mm, 8 parts, among them J1 1mm Pitch FPC, J2 0.8mm Pitch FPC, J3 0.5mm Pitch FPC, J4 JST-PH-3PIN, U1 SC0918

Commit message: Add files via upload
Parts:
- added J5, J6: JST-PH-2PIN, JST-PH-2PIN:JST-PH-2PIN
Connections:
- new net N$1: J5.P$2, U1.30
- new net N$2: J6.P$2, U1.37
- net GND: now also J5.P$1, J6.P$1
Routing:
- net N$2: track 0.00 -> 33.3 mm
- net N$1: track 0.00 -> 28.2 mm
- net GND: track 77.7 -> 74.1 mm
Other:
- board text added: "5V"
- board text added: "EN"
- board text added: "GND"
- board text added: "RST*"
- board text added: "Reset"
- board text added: "Shut Off"
- board text added: "VBAT"
Changed lines of the file:
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@@
 <drawing>
 <settings>
-<setting alwaysvectorfont="yes"/>
+<setting alwaysvectorfont="no"/>
 <setting verticaltext="up"/>
 </settings>
@@
 <wire x1="12" y1="0" x2="0" y2="0" width="0" layer="20"/>
 <text x="34.5" y="52.8" size="0.6096" layer="21" ratio="15">Battery</text>
-<text x="5.9" y="12.8" size="1.778" layer="21" ratio="15" rot="R90">Raspberry Pi Pico W
+<text x="36.86" y="9.66" size="1.778" layer="21" ratio="15" rot="R90">Raspberry Pi Pico W
 26 Pin Keyboard Controller</text>
+<text x="1.61" y="45.41" size="0.6096" layer="21" ratio="15">Shut Off</text>
+<text x="2.04" y="24.77" size="0.6096" layer="21" ratio="15">Reset</text>
+<text x="40.83" y="48.87" size="1.778" layer="22" rot="MR270">GND</text>
+<text x="42.81" y="48.89" size="1.778" layer="22" rot="MR270">5V</text>
+<text x="44.84" y="48.89" size="1.778" layer="22" rot="MR270">VBAT</text>
+<text x="4.95" y="44.21" size="1.778" layer="22" rot="MR0">EN</text>
+<text x="5.8" y="38.23" size="1.778" layer="22" rot="MR0">GND</text>
+<text x="6.01" y="17.65" size="1.778" layer="22" rot="MR0">GND</text>
+<text x="6.32" y="23.67" size="1.778" layer="22" rot="MR0">RST*</text>
 </plain>
 <attributes>
@@
 </element>
 <element name="J4" library="JST-PH-3PIN" package="JST-PH-3PIN" value="JST-PH-3PIN" x="42.9" y="51.1" smashed="yes">
-<attribute name="NAME" x="46.42" y="52.91" size="0.6096" layer="25"/>
+<attribute name="NAME" x="46.23" y="51.71" size="0.8128" layer="25"/>
 <attribute name="VALUE" x="39.32" y="53.01" size="0.6096" layer="27"/>
 </element>
@@
 <element name="U$1" library="oshw_revA" package="OSHW_8MM" value="" x="45.16" y="8.81" smashed="yes"/>
 <element name="U$2" library="oshw_backside" package="OSHW_8MM" value="" x="45.23" y="8.6" smashed="yes"/>
+<element name="J5" library="JST-PH-2PIN" package="JST-PH-2PIN" value="JST-PH-2PIN" x="3.35" y="21.44" smashed="yes" rot="R90">
+<attribute name="NAME" x="3.66" y="17.9" size="0.8128" layer="25" rot="R180"/>
+<attribute name="VALUE" x="5.62" y="19.14" size="0.6096" layer="27" rot="R90"/>
+</element>
+<element name="J6" library="JST-PH-2PIN" package="JST-PH-2PIN" value="JST-PH-2PIN" x="3.37" y="41.95" smashed="yes" rot="R90">
+<attribute name="NAME" x="3.64" y="38.38" size="0.8128" layer="25" rot="R180"/>
+<attribute name="VALUE" x="5.66" y="39.98" size="0.6096" layer="27" rot="R90"/>
+</element>
 </elements>
 <signals>
@@
 <via x="31.75" y="33.18" extent="1-16" drill="0.35"/>
 <wire x1="28.69" y1="33.15" x2="14.95" y2="33.15" width="1.27" layer="1"/>
-<wire x1="11.06" y1="37.04" x2="2.83" y2="37.04" width="0.1524" layer="1"/>
-<wire x1="2.83" y1="37.04" x2="2.83" y2="37.05" width="0.1524" layer="1"/>
-<via x="2.83" y="37.05" extent="1-16" drill="0.35"/>
+<wire x1="11.06" y1="37.04" x2="6.46" y2="37.04" width="0.1524" layer="1"/>
+<wire x1="6.46" y1="37.04" x2="6.46" y2="37.02" width="0.1524" layer="1"/>
+<via x="6.46" y="37.02" extent="1-16" drill="0.35"/>
 <wire x1="14.95" y1="33.15" x2="11.06" y2="37.04" width="0.1524" layer="1"/>
 <wire x1="28.69" y1="20.45" x2="30.29" y2="20.45" width="0.1524" layer="1"/>
@@
 <via x="31.12" y="8.19" extent="1-16" drill="0.35"/>
 <wire x1="30.54" y1="7.75" x2="30.98" y2="8.19" width="0.6096" layer="1"/>
+<contactref element="J5" pad="P$1"/>
+<contactref element="J6" pad="P$1"/>
 </signal>
 <signal name="ADC_VREF">
@@
 <wire x1="44.7" y1="35.1" x2="39.9" y2="37" width="0.1524" layer="1"/>
 <wire x1="37.6" y1="37" x2="38.74" y2="37" width="0.1524" layer="1"/>
-<wire x1="9.31" y1="48.39" x2="11.91" y2="48.39" width="0.1524" layer="1"/>
-<wire x1="11.91" y1="48.39" x2="14.88" y2="45.42" width="0.1524" layer="1"/>
-<wire x1="26.78" y1="42" x2="30.76" y2="42" width="0.1524" layer="1"/>
-<wire x1="14.88" y1="45.42" x2="23.36" y2="45.42" width="0.1524" layer="1"/>
-<wire x1="23.36" y1="45.42" x2="26.78" y2="42" width="0.1524" layer="1"/>
+<wire x1="9.31" y1="48.39" x2="11.5" y2="48.39" width="0.1524" layer="1"/>
+<wire x1="11.5" y1="48.39" x2="15.13" y2="44.76" width="0.1524" layer="1"/>
+<wire x1="23.99" y1="42" x2="30.76" y2="42" width="0.1524" layer="1"/>
+<wire x1="15.13" y1="44.76" x2="21.23" y2="44.76" width="0.1524" layer="1"/>
+<wire x1="21.23" y1="44.76" x2="23.99" y2="42" width="0.1524" layer="1"/>
 <wire x1="30.76" y1="42" x2="37.6" y2="37" width="0.1524" layer="1"/>
 </signal>
@@
 <wire x1="38.74" y1="36" x2="37.6" y2="36" width="0.1524" layer="1"/>
 <wire x1="9.31" y1="43.31" x2="12.02" y2="43.31" width="0.1524" layer="1"/>
-<wire x1="12.02" y1="43.31" x2="13.42" y2="44.71" width="0.1524" layer="1"/>
-<wire x1="13.42" y1="44.71" x2="19.65" y2="44.71" width="0.1524" layer="1"/>
-<wire x1="19.65" y1="44.71" x2="24.92" y2="39.44" width="0.1524" layer="1"/>
+<wire x1="12.02" y1="43.31" x2="12.87" y2="44.16" width="0.1524" layer="1"/>
+<wire x1="12.87" y1="44.16" x2="20.2" y2="44.16" width="0.1524" layer="1"/>
+<wire x1="20.2" y1="44.16" x2="24.92" y2="39.44" width="0.1524" layer="1"/>
 <wire x1="30.83" y1="39.44" x2="24.92" y2="39.44" width="0.1524" layer="1"/>
 <wire x1="37.6" y1="36" x2="30.83" y2="39.44" width="0.1524" layer="1"/>
@@
 <wire x1="37.6" y1="13" x2="30.85" y2="2.67" width="0.1524" layer="1"/>
 </signal>
+<signal name="N$1">
+<contactref element="J5" pad="P$2"/>
+<contactref element="U1" pad="30"/>
+<wire x1="3.35" y1="22.44" x2="5.6" y2="24.69" width="0.1524" layer="1"/>
+<wire x1="5.6" y1="24.69" x2="5.6" y2="25.69" width="0.1524" layer="1"/>
+<wire x1="5.6" y1="25.69" x2="6.7" y2="26.79" width="0.1524" layer="1"/>
+<wire x1="6.7" y1="26.79" x2="24.19" y2="26.79" width="0.1524" layer="1"/>
+<wire x1="25.45" y1="25.53" x2="24.19" y2="26.79" width="0.1524" layer="1"/>
+<wire x1="28.69" y1="25.53" x2="25.45" y2="25.53" width="0.1524" layer="1"/>
+</signal>
+<signal name="N$2">
+<contactref element="J6" pad="P$2"/>
+<contactref element="U1" pad="37"/>
+<wire x1="3.37" y1="42.95" x2="3.37" y2="47.28" width="0.1524" layer="1"/>
+<wire x1="5.76" y1="49.67" x2="11.12" y2="49.67" width="0.1524" layer="1"/>
+<wire x1="11.12" y1="49.67" x2="15.33" y2="45.46" width="0.1524" layer="1"/>
+<wire x1="25.71" y1="43.31" x2="26.73" y2="43.31" width="0.1524" layer="1"/>
+<wire x1="3.37" y1="47.28" x2="5.76" y2="49.67" width="0.1524" layer="1"/>
+<wire x1="15.33" y1="45.46" x2="23.56" y2="45.46" width="0.1524" layer="1"/>
+<wire x1="23.56" y1="45.46" x2="25.71" y2="43.31" width="0.1524" layer="1"/>
+<wire x1="28.69" y1="43.31" x2="26.73" y2="43.31" width="0.1524" layer="1"/>
+</signal>
 </signals>
