File: Example_Keyboards/Pico_26Pin_Keyboard/Pico_26Pin_Keyboard.sch (EAGLE design)
At the start: 6 parts, among them J1 1mm Pitch FPC, J2 0.8mm Pitch FPC, J3 0.5mm Pitch FPC, J4 JST-PH-3PIN, U1 SC0918

Commit message: Add files via upload
Parts:
- added J5, J6: JST-PH-2PIN, JST-PH-2PIN:JST-PH-2PIN
Connections:
- new net N$1: J5.P2, U1.RUN
- new net N$2: J6.P2, U1.3V3_EN
- net GND: now also J5.P1, J6.P1
Other:
- note added: "Install diode only if running from battery power"
- note added: "Wire to a Reset Push Button Switch"
- note added: "Wire to a Switch that powers down the Pico if running from a battery"
Changed lines of the file:
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@@
 <drawing>
 <settings>
-<setting alwaysvectorfont="yes"/>
+<setting alwaysvectorfont="no"/>
 <setting verticaltext="up"/>
 </settings>
@@
 <part name="J2" library="FPC26_p8mm" deviceset="FPC26_P8MM" device="" value="0.8mm Pitch FPC"/>
 <part name="J3" library="FPC26_p5mm" deviceset="FPC26_P5MM" device="" value="0.5mm Pitch FPC"/>
+<part name="J5" library="JST-PH-2PIN" deviceset="JST-PH-2PIN" device="" value="JST-PH-2PIN"/>
+<part name="SUPPLY2" library="supply2" library_urn="urn:adsk.eagle:library:372" deviceset="GND" device=""/>
+<part name="J6" library="JST-PH-2PIN" deviceset="JST-PH-2PIN" device="" value="JST-PH-2PIN"/>
+<part name="SUPPLY3" library="supply2" library_urn="urn:adsk.eagle:library:372" deviceset="GND" device=""/>
 </parts>
 <sheets>
 <sheet>
 <plain>
-<text x="-17.78" y="116.84" size="1.778" layer="97">Wire USB 5 Volts on pin 2 to a battery charger.
+<text x="-12.7" y="114.3" size="1.778" layer="97">Wire USB 5 Volts on pin 2 to a battery charger.
 Wire battery output to pin 3</text>
+<text x="-83.82" y="111.76" size="1.778" layer="97">Wire to a Reset Push Button Switch</text>
+<text x="-43.18" y="101.6" size="1.778" layer="97">Wire to a Switch that powers down the
+Pico if running from a battery</text>
+<text x="17.78" y="81.28" size="1.778" layer="97">Install diode only if running
+from battery power</text>
 </plain>
 <instances>
@@
 <attribute name="NAME" x="127" y="71.12" size="1.6764" layer="95"/>
 <attribute name="VALUE" x="119.38" y="-2.54" size="1.778" layer="96"/>
+</instance>
+<instance part="J5" gate="G$1" x="-55.88" y="102.362" smashed="yes" rot="R90">
+<attribute name="NAME" x="-63.5" y="102.362" size="1.778" layer="95" rot="R90"/>
+<attribute name="VALUE" x="-62.738" y="109.22" size="1.778" layer="96"/>
+</instance>
+<instance part="SUPPLY2" gate="GND" x="-58.42" y="88.9" smashed="yes">
+<attribute name="VALUE" x="-60.325" y="85.725" size="1.778" layer="96"/>
+</instance>
+<instance part="J6" gate="G$1" x="-22.86" y="92.202" smashed="yes" rot="R90">
+<attribute name="NAME" x="-30.48" y="92.202" size="1.778" layer="95" rot="R90"/>
+<attribute name="VALUE" x="-29.718" y="99.06" size="1.778" layer="96"/>
+</instance>
+<instance part="SUPPLY3" gate="GND" x="-25.4" y="78.74" smashed="yes">
+<attribute name="VALUE" x="-27.305" y="75.565" size="1.778" layer="96"/>
 </instance>
 </instances>
@@
 <wire x1="5.08" y1="93.98" x2="5.08" y2="96.52" width="0.1524" layer="91"/>
 </segment>
+<segment>
+<pinref part="J5" gate="G$1" pin="P1"/>
+<pinref part="SUPPLY2" gate="GND" pin="GND"/>
+<wire x1="-58.42" y1="94.742" x2="-58.42" y2="91.44" width="0.1524" layer="91"/>
+</segment>
+<segment>
+<pinref part="SUPPLY3" gate="GND" pin="GND"/>
+<pinref part="J6" gate="G$1" pin="P1"/>
+<wire x1="-25.4" y1="81.28" x2="-25.4" y2="84.582" width="0.1524" layer="91"/>
+</segment>
 </net>
 <net name="VSYS" class="0">
@@
 </segment>
 </net>
+<net name="N$1" class="0">
+<segment>
+<pinref part="J5" gate="G$1" pin="P2"/>
+<wire x1="-53.34" y1="94.742" x2="-53.34" y2="53.34" width="0.1524" layer="91"/>
+<pinref part="U1" gate="G$1" pin="RUN"/>
+<wire x1="-53.34" y1="53.34" x2="-48.26" y2="53.34" width="0.1524" layer="91"/>
+</segment>
+</net>
+<net name="N$2" class="0">
+<segment>
+<pinref part="J6" gate="G$1" pin="P2"/>
+<wire x1="-20.32" y1="84.582" x2="-20.32" y2="71.12" width="0.1524" layer="91"/>
+<wire x1="-20.32" y1="71.12" x2="-50.8" y2="71.12" width="0.1524" layer="91"/>
+<wire x1="-50.8" y1="71.12" x2="-50.8" y2="55.88" width="0.1524" layer="91"/>
+<pinref part="U1" gate="G$1" pin="3V3_EN"/>
+<wire x1="-50.8" y1="55.88" x2="-48.26" y2="55.88" width="0.1524" layer="91"/>
+</segment>
+</net>
