File: Example_Keyboards/Pico_26Pin_Keyboard/Pico_26Pin_FPC_Adapter.brd (EAGLE design)
At the start: 55 x 55 mm, 8 parts, among them J4 JST-PH-3PIN, J5 JST-PH-2PIN, J6 JST-PH-2PIN, U1 SC0918

Commit message: Add files via upload
Parts:
- D1: value MBR120VLSFT1G -> 1N5817; device SamacSys_Parts:SODFL3616X98N -> SamacSys_Parts:DIOAD1410W86L470D235
- moved D1 2.21 mm to (33.0, 46.6)
Routing:
- net GND: track 71.1 -> 79.4 mm
- net VBAT: track 10.5 -> 7.66 mm
- net VSYS: track 4.23 -> 6.10 mm
Other:
- board text added: "1N5817"
Changed lines of the file:
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@@
 <wire x1="12" y1="0" x2="0" y2="0" width="0" layer="20"/>
 <text x="34.5" y="52.8" size="0.6096" layer="21" ratio="15">Battery</text>
-<text x="37.58" y="13.71" size="1.778" layer="21" ratio="15" rot="R90">Raspberry Pi Pico W
-26 Pin Keyboard Controller</text>
+<text x="37.77" y="12.82" size="1.778" layer="21" ratio="15" rot="R90">Raspberry Pi Pico W 26 Pin
+Keyboard Controller</text>
 <text x="1.61" y="45.41" size="0.6096" layer="21" ratio="15">Shut Off</text>
 <text x="2.04" y="24.77" size="0.6096" layer="21" ratio="15">Reset</text>
@@
 <text x="45.68" y="12.38" size="1.778" layer="21">23</text>
 <text x="45.69" y="9.77" size="1.778" layer="21">25</text>
+<text x="36.35" y="43.73" size="1.4224" layer="21">1N5817</text>
+<wire x1="40.73" y1="47.51" x2="40.73" y2="45.78" width="0.1524" layer="21"/>
+<wire x1="40.73" y1="45.78" x2="39.88" y2="46.63" width="0.1524" layer="21"/>
+<wire x1="39.88" y1="46.63" x2="39.88" y2="46.64" width="0.1524" layer="21"/>
+<wire x1="39.88" y1="46.64" x2="40.73" y2="47.49" width="0.1524" layer="21"/>
+<wire x1="40.73" y1="47.49" x2="40.74" y2="47.49" width="0.1524" layer="21"/>
+<wire x1="39.88" y1="47.52" x2="39.88" y2="45.75" width="0.1524" layer="21"/>
+<wire x1="39.88" y1="47.52" x2="39.87" y2="47.53" width="0.1524" layer="21"/>
+<wire x1="39.87" y1="47.53" x2="39.56" y2="47.53" width="0.1524" layer="21"/>
+<wire x1="39.56" y1="47.53" x2="39.56" y2="47.22" width="0.1524" layer="21"/>
+<wire x1="39.88" y1="45.75" x2="40.18" y2="45.75" width="0.1524" layer="21"/>
+<wire x1="40.18" y1="45.75" x2="40.18" y2="46.03" width="0.1524" layer="21"/>
 </plain>
 <attributes>
@@
 <attribute name="VALUE" x="15.76" y="12" size="1.27" layer="27" align="top-left"/>
 </element>
-<element name="D1" library="SamacSys_Parts" package="SODFL3616X98N" value="MBR120VLSFT1G" x="34.37" y="48.42" smashed="yes">
-<attribute name="DESCRIPTION" value="Diode Schottky 20V 1A SOD123FL ON Semi MBR120VLSFT1G, SMT Schottky Diode, 20V 1A, 2-Pin SOD-123FL" x="23.17" y="57.12" size="1.778" layer="27" display="off"/>
-<attribute name="HEIGHT" value="0.98mm" x="23.17" y="57.12" size="1.778" layer="27" display="off"/>
-<attribute name="MANUFACTURER_NAME" value="onsemi" x="23.17" y="57.12" size="1.778" layer="27" display="off"/>
-<attribute name="MANUFACTURER_PART_NUMBER" value="MBR120VLSFT1G" x="23.17" y="57.12" size="1.778" layer="27" display="off"/>
-<attribute name="MOUSER_PART_NUMBER" value="863-MBR120VLSFT1G" x="23.17" y="57.12" size="1.778" layer="27" display="off"/>
-<attribute name="MOUSER_PRICE-STOCK" value="https://www.mouser.co.uk/ProductDetail/onsemi/MBR120VLSFT1G?qs=3JMERSakebpX%252BkItPpFCkg%3D%3D" x="23.17" y="57.12" size="1.778" layer="27" display="off"/>
-<attribute name="NAME" x="34.37" y="45.88" size="1.27" layer="25" align="center"/>
-<attribute name="VALUE" x="34.37" y="52.23" size="1.27" layer="27" align="center"/>
+<element name="D1" library="SamacSys_Parts" package="DIOAD1410W86L470D235" value="1N5817" x="33.04" y="46.65" smashed="yes">
+<attribute name="DESCRIPTION" value="Schottky Diodes &amp; Rectifiers 1A, 20V, Schottky Rectifier" x="21.84" y="55.35" size="1.778" layer="27" display="off"/>
+<attribute name="HEIGHT" value="mm" x="21.84" y="55.35" size="1.778" layer="27" display="off"/>
+<attribute name="MANUFACTURER_NAME" value="Taiwan Semiconductor" x="21.84" y="55.35" size="1.778" layer="27" display="off"/>
+<attribute name="MANUFACTURER_PART_NUMBER" value="1N5817" x="21.84" y="55.35" size="1.778" layer="27" display="off"/>
+<attribute name="MOUSER_PART_NUMBER" value="821-1N5817" x="21.84" y="55.35" size="1.778" layer="27" display="off"/>
+<attribute name="MOUSER_PRICE-STOCK" value="https://www.mouser.co.uk/ProductDetail/Taiwan-Semiconductor/1N5817?qs=G5AQjGfRJcITga2hz4Rc2w%3D%3D" x="21.84" y="55.35" size="1.778" layer="27" display="off"/>
+<attribute name="NAME" x="36.43" y="48.08" size="1.27" layer="25" align="center"/>
+<attribute name="VALUE" x="33.04" y="50.46" size="1.27" layer="27" align="center"/>
 </element>
 <element name="J4" library="JST-PH-3PIN" package="JST-PH-3PIN" value="JST-PH-3PIN" x="42.9" y="51.1" smashed="yes">
@@
 </element>
 <element name="J1" library="SparkFun-Connectors" package="2X13" package3d_urn="urn:adsk.eagle:package:38269/1" value="" x="41.24" y="41.16" smashed="yes" rot="R270">
-<attribute name="NAME" x="43.144" y="43.66" size="0.6096" layer="25" font="vector" ratio="20" rot="R270"/>
+<attribute name="NAME" x="44.194" y="43.66" size="0.6096" layer="25" font="vector" ratio="20" rot="R270"/>
 <attribute name="VALUE" x="38.827" y="42.43" size="0.6096" layer="27" font="vector" ratio="20" rot="R270"/>
 </element>
@@
 <wire x1="28.64" y1="20.45" x2="28.69" y2="20.45" width="0.1524" layer="1"/>
 <contactref element="J4" pad="P$1"/>
-<wire x1="26.9" y1="20.45" x2="28.64" y2="20.45" width="1.27" layer="1"/>
+<wire x1="26.9" y1="20.45" x2="27.8" y2="20.45" width="1.27" layer="1"/>
+<wire x1="27.8" y1="20.45" x2="28.64" y2="20.45" width="1.27" layer="1"/>
 <wire x1="10.11" y1="20.45" x2="16.35" y2="20.45" width="1.27" layer="1"/>
 <wire x1="16.35" y1="20.45" x2="17.75" y2="19.05" width="1.27" layer="1"/>
@@
 <wire x1="10.11" y1="45.85" x2="9.38" y2="45.85" width="1.27" layer="1"/>
 <wire x1="9.31" y1="45.85" x2="6.23" y2="45.85" width="1.27" layer="1"/>
-<wire x1="27.89" y1="45.85" x2="28.69" y2="45.85" width="1.27" layer="1"/>
+<wire x1="27.89" y1="45.85" x2="28.44" y2="45.85" width="1.27" layer="1"/>
+<wire x1="28.44" y1="45.85" x2="28.69" y2="45.85" width="1.27" layer="1"/>
 <wire x1="28.69" y1="33.15" x2="31.72" y2="33.15" width="1.27" layer="1"/>
 <wire x1="31.72" y1="33.15" x2="31.75" y2="33.18" width="1.27" layer="1"/>
@@
 <contactref element="J5" pad="P$1"/>
 <contactref element="J6" pad="P$1"/>
+<wire x1="31.38" y1="7.72" x2="28.27" y2="7.72" width="1.27" layer="1"/>
+<wire x1="30.91" y1="20.45" x2="28.64" y2="20.45" width="1.27" layer="1"/>
+<wire x1="31.36" y1="45.83" x2="28.46" y2="45.83" width="1.27" layer="1"/>
+<wire x1="28.46" y1="45.83" x2="28.44" y2="45.85" width="1.27" layer="1"/>
 </signal>
 <signal name="ADC_VREF">
@@
 <contactref element="U1" pad="39"/>
 <wire x1="29.0764" y1="48.42" x2="29.0464" y2="48.39" width="0.508" layer="1"/>
-<wire x1="32.84" y1="48.39" x2="32.87" y2="48.42" width="0.508" layer="1"/>
-<wire x1="28.69" y1="48.39" x2="32.84" y2="48.39" width="1.016" layer="1"/>
+<wire x1="33.04" y1="46.65" x2="33.00588125" y2="48.39" width="1.016" layer="1"/>
+<wire x1="28.69" y1="48.39" x2="33.00588125" y2="48.39" width="1.016" layer="1"/>
 <wire x1="28.69" y1="48.39" x2="29.0464" y2="48.39" width="0" layer="19" extent="1-1"/>
 </signal>
@@
 <contactref element="D1" pad="2"/>
 <contactref element="J4" pad="P$3"/>
-<wire x1="35.87" y1="48.42" x2="43.43" y2="48.42" width="1.016" layer="1"/>
-<wire x1="43.43" y1="48.42" x2="43.96" y2="48.95" width="1.016" layer="1"/>
-<wire x1="43.96" y1="48.95" x2="43.96" y2="51.07" width="1.016" layer="1"/>
+<wire x1="47.14" y1="46.65" x2="43.96" y2="46.65" width="1.016" layer="1"/>
+<wire x1="43.96" y1="46.65" x2="43.96" y2="51.07" width="1.016" layer="1"/>
 <wire x1="43.96" y1="51.07" x2="43.92" y2="51.11" width="0.508" layer="1"/>
 </signal>
@@
 <wire x1="26.4572" y1="10.48938125" x2="26.4572" y2="6.6" width="0.1524" layer="1"/>
 <wire x1="26.4572" y1="6.6" x2="26.5572" y2="6.5" width="0.1524" layer="1"/>
-<wire x1="30.67" y1="6.5" x2="26.5572" y2="6.5" width="0.1524" layer="1"/>
+<wire x1="31.51" y1="6.5" x2="26.5572" y2="6.5" width="0.1524" layer="1"/>
 <wire x1="11.8" y1="10.8" x2="26.14658125" y2="10.8" width="0.1524" layer="1"/>
 <wire x1="26.14658125" y1="10.8" x2="26.4572" y2="10.48938125" width="0.1524" layer="1"/>
@@
 <wire x1="9.34" y1="2.7" x2="11.3" y2="2.7" width="0.1524" layer="1"/>
 <contactref element="J1" pad="23"/>
-<wire x1="30.67" y1="6.5" x2="37.39" y2="13.22" width="0.1524" layer="1"/>
-<wire x1="37.39" y1="13.22" x2="41.24" y2="13.22" width="0.1524" layer="1"/>
+<wire x1="31.51" y1="6.5" x2="38.23" y2="13.22" width="0.1524" layer="1"/>
+<wire x1="38.23" y1="13.22" x2="41.24" y2="13.22" width="0.1524" layer="1"/>
 </signal>
 <signal name="17">
