File: Example_Keyboards/Pico_26Pin_Keyboard/Pico_26Pin_FPC_Adapter.sch (EAGLE design)
At the start: 6 parts, among them J4 JST-PH-3PIN, J5 JST-PH-2PIN, J6 JST-PH-2PIN, U1 SC0918

Commit message: Add files via upload
Parts:
- D1: value MBR120VLSFT1G -> 1N5817; device SamacSys_Parts:MBR120VLSFT1G -> SamacSys_Parts:1N5817
Changed lines of the file:
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@@
 <part name="U1" library="SC0918" deviceset="SC0918" device=""/>
 <part name="SUPPLY1" library="supply2" library_urn="urn:adsk.eagle:library:372" deviceset="GND" device=""/>
-<part name="D1" library="SamacSys_Parts" deviceset="MBR120VLSFT1G" device=""/>
+<part name="D1" library="SamacSys_Parts" deviceset="1N5817" device=""/>
 <part name="SUPPLY5" library="supply2" library_urn="urn:adsk.eagle:library:372" deviceset="GND" device=""/>
 <part name="J4" library="JST-PH-3PIN" deviceset="JST-PH-3PIN" device="" value="JST-PH-3PIN"/>
@@
 </instance>
 <instance part="D1" gate="G$1" x="10.16" y="71.12" smashed="yes" rot="R90">
-<attribute name="NAME" x="12.7" y="82.55" size="1.778" layer="95" rot="R90" align="center-left"/>
-<attribute name="VALUE" x="15.24" y="72.39" size="1.778" layer="96" rot="R90" align="center-left"/>
+<attribute name="NAME" x="12.7" y="85.09" size="1.778" layer="95" rot="R90" align="center-left"/>
+<attribute name="VALUE" x="15.24" y="77.47" size="1.778" layer="96" rot="R90" align="center-left"/>
 </instance>
 <instance part="SUPPLY5" gate="GND" x="5.08" y="91.44" smashed="yes">
@@
 <net name="VSYS" class="0">
 <segment>
-<wire x1="10.16" y1="58.42" x2="10.16" y2="71.12" width="0.1524" layer="91"/>
+<wire x1="10.16" y1="58.42" x2="10.16" y2="73.66" width="0.1524" layer="91"/>
 <pinref part="D1" gate="G$1" pin="K"/>
 <pinref part="U1" gate="G$1" pin="VSYS"/>
@@
 <net name="VBAT" class="0">
 <segment>
-<wire x1="10.16" y1="86.36" x2="10.16" y2="96.52" width="0.1524" layer="91"/>
+<wire x1="10.16" y1="88.9" x2="10.16" y2="96.52" width="0.1524" layer="91"/>
 <pinref part="D1" gate="G$1" pin="A"/>
 <pinref part="J4" gate="G$1" pin="P3"/>
